Commit message: endrer variabler

File: src/tht_robot_env/urdf/ur_macro_pointer.xacro (robot description, xacro)
@@ -335,5 +335,5 @@
     <joint name="tool0-pointer" type="fixed">
       <!-- default toolframe - X+ left, Y+ up, Z+ front -->
-      <origin xyz="0 ${offset} 0.0850" rpy="0 0 0"/>
+      <origin xyz="0 ${offset} 0" rpy="0 0 0"/>
       <parent link="${prefix}tool0"/>
       <child link="pointer_tool"/>
