Commit message: working launch file for different end-effectors

File: src/tht_robot_env/urdf/ur_macro_test.xacro (robot description, xacro)
@@ -319,45 +319,48 @@
     <xacro:property name="offset" value="0"/>
     <!-- VETLE TEST -->
-    <link name="end_effector_1">
-      <visual>
-        <origin xyz="0 0 0" rpy="0 0 0"/>
-        <geometry>
-          <mesh filename="package://tht_robot_env/meshes/camera_calib_A4_Tool.stl" scale="0.001 0.001 0.001"/>
-        </geometry>
-        <material name="black"/>
-      </visual>
-      <collision>
-        <origin xyz="0 0 0" rpy="0 0 0"/>
-        <geometry>
-          <mesh filename="package://tht_robot_env/meshes/camera_calib_A4_Tool.stl"  scale="0.001 0.001 0.001"/>
-        </geometry>
-      </collision>
-    </link>
-    <link name="end_effector_2">
-      <visual>
-        <origin xyz="0 0 0" rpy="0 0 0"/>
-        <geometry>
-          <mesh filename="package://tht_robot_env/meshes/pointer_tool.stl" scale="0.001 0.001 0.001"/>
-        </geometry>
-        <material name="blue"/>
-      </visual>
-      <collision>
-        <origin xyz="0 0 0" rpy="0 0 0"/>
-        <geometry>
-          <mesh filename="package://tht_robot_env/meshes/pointer_tool.stl"  scale="0.001 0.001 0.001"/>
-        </geometry>
-      </collision>
-    </link>
-    <joint name="end_effector_joint" type="fixed">
-      <parent link="tool0"/>
-      <xacro:if value="${end_effector_type == 1}">
+    <xacro:if value="${end_effector_type == 1}">
+      <link name="end_effector_1">
+        <visual>
+          <origin xyz="0 0 0" rpy="0 0 0"/>
+          <geometry>
+            <mesh filename="package://tht_robot_env/meshes/camera_calib_A4_Tool.stl" scale="0.001 0.001 0.001"/>
+          </geometry>
+          <material name="black"/>
+        </visual>
+        <collision>
+          <origin xyz="0 0 0" rpy="0 0 0"/>
+          <geometry>
+            <mesh filename="package://tht_robot_env/meshes/camera_calib_A4_Tool.stl"  scale="0.001 0.001 0.001"/>
+          </geometry>
+        </collision>
+      </link>
+      <joint name="end_effector_joint" type="fixed">
+        <parent link="tool0"/>
         <origin xyz="0 0 0.0850" rpy="0 0 0"/>
         <child link="end_effector_1"/>
-      </xacro:if>
-      <xacro:if value="${end_effector_type == 2}">
-        <origin xyz="0 0 0.0850" rpy="0 0 0"/>
+      </joint>
+    </xacro:if>
+    <xacro:if value="${end_effector_type == 2}">
+      <link name="end_effector_2">
+        <visual>
+          <origin xyz="0 0 0" rpy="0 0 0"/>
+          <geometry>
+            <mesh filename="package://tht_robot_env/meshes/pointer_tool.stl" scale="0.001 0.001 0.001"/>
+          </geometry>
+          <material name="white"/>
+        </visual>
+        <collision>
+          <origin xyz="0 0 0" rpy="0 0 0"/>
+          <geometry>
+            <mesh filename="package://tht_robot_env/meshes/pointer_tool.stl"  scale="0.001 0.001 0.001"/>
+          </geometry>
+        </collision>
+      </link>
+      <joint name="end_effector_joint" type="fixed">
+        <origin xyz="0 0 0.133" rpy="0 0 0"/>
         <child link="end_effector_2"/>
-      </xacro:if>
-    </joint>
+        <parent link="tool0"/>
+      </joint>
+    </xacro:if>
     <link name="ground">
 		<visual>
