Commit message: Rotated OAK camera axes with new link

File: src/tht_robot_env/urdf/inc/cameras/fixed_camera_cameracalib.xacro (robot description, xacro)
@@ -27,4 +27,16 @@
       		<child link="OAK_camera" />
 	</joint>
+	<!-- ROS-Industrial 'base' frame - base_link to UR 'Base' Coordinates transform -->
+    <link name="OAK_camera_rot"/>
+    <joint name="OAK_link-OAK_fixed_joint" type="fixed">
+      <!-- Note the rotation over Z of pi radians - as base_link is REP-103
+           aligned (i.e., has X+ forward, Y+ left and Z+ up), this is needed
+           to correctly align 'base' with the 'Base' coordinate system of
+           the UR controller.
+      -->
+      <origin xyz="0 0 0" rpy="${-pi/2} 0 0"/>
+      <parent link="OAK_camera"/>
+      <child link="OAK_camera_rot"/>
+    </joint>
 	<link name="camera_stand">
 		<visual>

File: src/tht_robot_env/urdf/ur_macro_cameracalib.xacro (robot description, xacro)
@@ -335,5 +335,5 @@
     <joint name="tool0-calib" type="fixed">
       <!-- default toolframe - X+ left, Y+ up, Z+ front -->
-      <origin xyz="0 ${offset} 0" rpy="0 0 0"/>
+      <origin xyz="0 ${offset} 0.0850" rpy="0 0 0"/>
       <parent link="${prefix}tool0"/>
       <child link="calib_board"/>
