Commit message: remove logs and changed pkg name

File: src/tht_robot_env/urdf/inc/cameras/fixed_camera.xacro (robot description, xacro)
@@ -2,5 +2,5 @@
 <robot xmlns:xacro="http://wiki.ros.org/xacro">
 	<!-- Create yaml file with measurements for the fixed_gripper-->
-	<xacro:property name="file"    value="$(find thtr_robot_env)/urdf/inc/cameras/cam_info.yaml"/>
+	<xacro:property name="file"    value="$(find tht_robot_env)/urdf/inc/cameras/cam_info.yaml"/>
   <xacro:property name="measurements"   value="${xacro.load_yaml(file)}"/>
 	<!-- measurements for camera dimensions-->

File: src/tht_robot_env/urdf/inc/cameras/fixed_camera_bachelor.xacro (robot description, xacro)
@@ -2,10 +2,10 @@
 <robot xmlns:xacro="http://wiki.ros.org/xacro">
 	<!-- Create yaml file with measurements for the fixed_gripper-->
-	<xacro:property name="file"    value="$(find thtr_robot_env)/urdf/inc/cameras/cam_info.yaml"/>
+	<xacro:property name="file"    value="$(find tht_robot_env)/urdf/inc/cameras/cam_info.yaml"/>
   <xacro:property name="measurements"   value="${xacro.load_yaml(file)}"/>
 	<!-- measurements for camera dimensions-->
   <xacro:property name="camera" value="${measurements['dimensions']}"/>
   <!-- Create yaml file with calibration transform for the fixed camera-->
-	<xacro:property name="file"    value="$(find thtr_robot_env)/urdf/inc/cameras/easy_handeye_eye_on_base.yaml"/>
+	<xacro:property name="file"    value="$(find tht_robot_env)/urdf/inc/cameras/easy_handeye_eye_on_base.yaml"/>
   <xacro:property name="cali_measurements"   value="${xacro.load_yaml(file)}"/>
   <!-- measurements for camera coordinates-->

File: src/tht_robot_env/urdf/inc/cameras/fixed_camera_cameracalib.xacro (robot description, xacro)
@@ -2,5 +2,5 @@
 <robot xmlns:xacro="http://wiki.ros.org/xacro">
 	<!-- Create yaml file with measurements for the fixed_gripper-->
-	<xacro:property name="file"    value="$(find thtr_robot_env)/urdf/inc/cameras/cam_info_cameracalib.yaml"/>
+	<xacro:property name="file"    value="$(find tht_robot_env)/urdf/inc/cameras/cam_info_cameracalib.yaml"/>
   <xacro:property name="measurements"   value="${xacro.load_yaml(file)}"/>
 	<!-- measurements for camera dimensions-->

File: src/tht_robot_env/urdf/inc/cameras/gripper_camera.xacro (robot description, xacro)
@@ -2,5 +2,5 @@
 <robot xmlns:xacro="http://wiki.ros.org/xacro">
 	<xacro:macro name="gripper_cam" params="base">
-		<xacro:property name="file" value="$(find thtr_robot_env)/urdf/inc/cameras/cam_info.yaml"/>
+		<xacro:property name="file" value="$(find tht_robot_env)/urdf/inc/cameras/cam_info.yaml"/>
   	<xacro:property name="measurements" value="${xacro.load_yaml(file)}"/>
 		<!-- measurements for camera dimensions-->

File: src/tht_robot_env/urdf/inc/workspace_macro.xacro (robot description, xacro)
@@ -30,5 +30,5 @@
     		<origin xyz= "${origin_xyz}" rpy ="${origin_rpy}"/>
     		<geometry>
-    			<mesh filename="package://thtr_robot_env/meshes/crate.dae"/>
+    			<mesh filename="package://tht_robot_env/meshes/crate.dae"/>
     		</geometry>
     		<material name="green"/>
@@ -37,5 +37,5 @@
     		<origin xyz= "${origin_xyz}" rpy ="${origin_rpy}"/>
     		<geometry>
-    			<mesh filename="package://thtr_robot_env/meshes/crate.dae"/>
+    			<mesh filename="package://tht_robot_env/meshes/crate.dae"/>
     		</geometry>
     	</collision>

File: src/tht_robot_env/urdf/inc/workspaces/space2_desc.xacro (robot description, xacro)
@@ -4,6 +4,6 @@
 <xacro:macro name="space2" params="base">
  <!-- including the workspace macro -->
-    <xacro:include filename="$(find thtr_robot_env)/urdf/inc/workspaces/workspace_macro.xacro" />
-    <xacro:property name="value_file"    value="$(find thtr_robot_env)/urdf/inc/workspaces/space2.yaml" />
+    <xacro:include filename="$(find tht_robot_env)/urdf/inc/workspaces/workspace_macro.xacro" />
+    <xacro:property name="value_file"    value="$(find tht_robot_env)/urdf/inc/workspaces/space2.yaml" />
     <xacro:property name="measurements"   value="${xacro.load_yaml(value_file)}" />
     <!-- measurements and parameters for robot_table-->
@@ -13,5 +13,5 @@
     <!-- measurements and parameters for crates-->
     <xacro:property name="crates" value="${measurements['crate_dimensions']}"/>
-    <xacro:property name="tags_value_file"    value="$(find thtr_robot_env)/urdf/inc/workspaces/tag_coords.yaml" />
+    <xacro:property name="tags_value_file"    value="$(find tht_robot_env)/urdf/inc/workspaces/tag_coords.yaml" />
     <xacro:property name="yamlmeasurements"   value="${xacro.load_yaml(tags_value_file)}" />
     <!-- measurements and parameters for robot_table-->

File: src/tht_robot_env/urdf/inc/workspaces/workspace_macro.xacro (robot description, xacro)
@@ -25,5 +25,5 @@
     		<origin xyz= "0 0 0" rpy ="${pi/2.0} 0 ${pi/2.0}"/>
     		<geometry>
-    			<mesh filename="package://thtr_robot_env/meshes/crate.dae"/>
+    			<mesh filename="package://tht_robot_env/meshes/crate.dae"/>
     		</geometry>
     	</visual>
@@ -31,5 +31,5 @@
     		<origin xyz= "0 0 0" rpy ="${pi/2.0} 0 ${pi/2.0}"/>
     		<geometry>
-    			<mesh filename="package://thtr_robot_env/meshes/crate.dae"/>
+    			<mesh filename="package://tht_robot_env/meshes/crate.dae"/>
     		</geometry>
     	</collision>

File: src/tht_robot_env/urdf/testur.urdf.xacro (robot description, xacro)
@@ -3,13 +3,13 @@
    <!-- robot name parameter -->
    <!-- import main macro -->
-   <xacro:include filename="$(find thtr_robot_env)/urdf/ur_macro.xacro"/>
+   <xacro:include filename="$(find tht_robot_env)/urdf/ur_macro.xacro"/>
    <!-- arm -->
    <xacro:ur_robot
      prefix=""
      parent="world"
-     joint_limits_parameters_file="$(find thtr_robot_env)/config/ur10e/joint_limits.yaml"
-     kinematics_parameters_file="$(find thtr_robot_env)/config/ur10e/default_kinematics.yaml"
-     physical_parameters_file="$(find thtr_robot_env)/config/ur10e/physical_parameters.yaml"
-     visual_parameters_file="$(find thtr_robot_env)/config/ur10e/visual_parameters.yaml"
+     joint_limits_parameters_file="$(find tht_robot_env)/config/ur10e/joint_limits.yaml"
+     kinematics_parameters_file="$(find tht_robot_env)/config/ur10e/default_kinematics.yaml"
+     physical_parameters_file="$(find tht_robot_env)/config/ur10e/physical_parameters.yaml"
+     visual_parameters_file="$(find tht_robot_env)/config/ur10e/visual_parameters.yaml"
      transmission_hw_interface=""
      safety_limits="false"

File: src/tht_robot_env/urdf/ur.urdf.cameracalib.xacro (robot description, xacro)
@@ -3,13 +3,13 @@
    <!-- robot name parameter -->
    <!-- import main macro -->
-   <xacro:include filename="$(find thtr_robot_env)/urdf/ur_macro_cameracalib.xacro"/>
+   <xacro:include filename="$(find tht_robot_env)/urdf/ur_macro_cameracalib.xacro"/>
    <!-- arm -->
    <xacro:ur_robot
      prefix=""
      parent="world"
-     joint_limits_parameters_file="$(find thtr_robot_env)/config/ur10e/joint_limits.yaml"
-     kinematics_parameters_file="$(find thtr_robot_env)/config/ur10e/default_kinematics.yaml"
-     physical_parameters_file="$(find thtr_robot_env)/config/ur10e/physical_parameters.yaml"
-     visual_parameters_file="$(find thtr_robot_env)/config/ur10e/visual_parameters.yaml"
+     joint_limits_parameters_file="$(find tht_robot_env)/config/ur10e/joint_limits.yaml"
+     kinematics_parameters_file="$(find tht_robot_env)/config/ur10e/default_kinematics.yaml"
+     physical_parameters_file="$(find tht_robot_env)/config/ur10e/physical_parameters.yaml"
+     visual_parameters_file="$(find tht_robot_env)/config/ur10e/visual_parameters.yaml"
      transmission_hw_interface=""
      safety_limits="false"

File: src/tht_robot_env/urdf/ur.urdf.pointer.xacro (robot description, xacro)
@@ -3,13 +3,13 @@
    <!-- robot name parameter -->
    <!-- import main macro -->
-   <xacro:include filename="$(find thtr_robot_env)/urdf/ur_macro_pointer.xacro"/>
+   <xacro:include filename="$(find tht_robot_env)/urdf/ur_macro_pointer.xacro"/>
    <!-- arm -->
    <xacro:ur_robot
      prefix=""
      parent="world"
-     joint_limits_parameters_file="$(find thtr_robot_env)/config/ur10e/joint_limits.yaml"
-     kinematics_parameters_file="$(find thtr_robot_env)/config/ur10e/default_kinematics.yaml"
-     physical_parameters_file="$(find thtr_robot_env)/config/ur10e/physical_parameters.yaml"
-     visual_parameters_file="$(find thtr_robot_env)/config/ur10e/visual_parameters.yaml"
+     joint_limits_parameters_file="$(find tht_robot_env)/config/ur10e/joint_limits.yaml"
+     kinematics_parameters_file="$(find tht_robot_env)/config/ur10e/default_kinematics.yaml"
+     physical_parameters_file="$(find tht_robot_env)/config/ur10e/physical_parameters.yaml"
+     visual_parameters_file="$(find tht_robot_env)/config/ur10e/visual_parameters.yaml"
      transmission_hw_interface=""
      safety_limits="false"

File: src/tht_robot_env/urdf/ur10e.urdf.xacro (robot description, xacro)
@@ -4,5 +4,5 @@
    <xacro:arg name="name" value="ur"/>
    <!-- import main macro -->
-   <xacro:include filename="$(find thtr_robot_env)/urdf/ur_macro.xacro"/>
+   <xacro:include filename="$(find tht_robot_env)/urdf/ur_macro.xacro"/>
    <!-- possible 'ur_type' values: ur3, ur3e, ur5, ur5e, ur10, ur10e, ur16e -->
    <!-- the default value should raise an error in case this was called without defining the type -->
@@ -41,5 +41,5 @@
    <xacro:arg name="simulation_controllers" value="" />
    <!-- initial position for simulations (Fake Hardware, Gazebo, Ignition) -->
-   <xacro:arg name="initial_positions_file" value="$(find thtr_robot_env)/config/initial_positions.yaml"/>
+   <xacro:arg name="initial_positions_file" value="$(find tht_robot_env)/config/initial_positions.yaml"/>
    <!-- convert to property to use substitution in function -->
    <xacro:property name="initial_positions_file" value="$(arg initial_positions_file)"/>

File: src/tht_robot_env/urdf/ur_macro.xacro (robot description, xacro)
@@ -1,6 +1,6 @@
 <?xml version="1.0"?>
 <robot xmlns:xacro="http://wiki.ros.org/xacro">
-  <xacro:include filename="$(find thtr_robot_env)/urdf/inc/ur_transmissions.xacro" />
-  <xacro:include filename="$(find thtr_robot_env)/urdf/inc/ur_common.xacro" />
+  <xacro:include filename="$(find tht_robot_env)/urdf/inc/ur_transmissions.xacro" />
+  <xacro:include filename="$(find tht_robot_env)/urdf/inc/ur_common.xacro" />
   <xacro:macro name="ur_robot" params="
     prefix
@@ -322,5 +322,5 @@
         <origin xyz="0 0 0" rpy="0 0 0"/>
         <geometry>
-          <mesh filename="package://thtr_robot_env/meshes/camera_calib_A4_Tool.stl" scale="0.001 0.001 0.001"/>
+          <mesh filename="package://tht_robot_env/meshes/camera_calib_A4_Tool.stl" scale="0.001 0.001 0.001"/>
         </geometry>
         <material name="black"/>
@@ -329,5 +329,5 @@
         <origin xyz="0 0 0" rpy="0 0 0"/>
         <geometry>
-          <mesh filename="package://thtr_robot_env/meshes/camera_calib_A4_Tool.stl"  scale="0.001 0.001 0.001"/>
+          <mesh filename="package://tht_robot_env/meshes/camera_calib_A4_Tool.stl"  scale="0.001 0.001 0.001"/>
         </geometry>
       </collision>
@@ -358,11 +358,11 @@
 	</joint>
     <!-- including the workspace urdf -->
-    <xacro:include filename="$(find thtr_robot_env)/urdf/inc/workspaces/space2_desc.xacro" />
+    <xacro:include filename="$(find tht_robot_env)/urdf/inc/workspaces/space2_desc.xacro" />
     <xacro:space2 base="${prefix}base_link"/>
     <!--Here another xacro:include for fixed_camera-->
-    <xacro:include filename="$(find thtr_robot_env)/urdf/inc/cameras/fixed_camera.xacro"/>
+    <xacro:include filename="$(find tht_robot_env)/urdf/inc/cameras/fixed_camera.xacro"/>
     <xacro:fixed_cam base="${prefix}base_link"/>
     <!--Here another xacro:include for gripper_camera-->
-    <!--xacro:include filename="$(find thtr_robot_env)/urdf/inc/cameras/gripper_camera.xacro"/>
+    <!--xacro:include filename="$(find tht_robot_env)/urdf/inc/cameras/gripper_camera.xacro"/>
     <xacro:gripper_cam base="${prefix}wrist_3_link"/-->
   </xacro:macro>

File: src/tht_robot_env/urdf/ur_macro_cameracalib.xacro (robot description, xacro)
@@ -1,6 +1,6 @@
 <?xml version="1.0"?>
 <robot xmlns:xacro="http://wiki.ros.org/xacro">
-  <xacro:include filename="$(find thtr_robot_env)/urdf/inc/ur_transmissions.xacro" />
-  <xacro:include filename="$(find thtr_robot_env)/urdf/inc/ur_common.xacro" />
+  <xacro:include filename="$(find tht_robot_env)/urdf/inc/ur_transmissions.xacro" />
+  <xacro:include filename="$(find tht_robot_env)/urdf/inc/ur_common.xacro" />
   <xacro:macro name="ur_robot" params="
     prefix
@@ -322,5 +322,5 @@
         <origin xyz="0 0 0" rpy="0 0 0"/>
         <geometry>
-          <mesh filename="package://thtr_robot_env/meshes/camera_calib_A4_Tool.stl" scale="0.001 0.001 0.001"/>
+          <mesh filename="package://tht_robot_env/meshes/camera_calib_A4_Tool.stl" scale="0.001 0.001 0.001"/>
         </geometry>
         <material name="black"/>
@@ -329,5 +329,5 @@
         <origin xyz="0 0 0" rpy="0 0 0"/>
         <geometry>
-          <mesh filename="package://thtr_robot_env/meshes/camera_calib_A4_Tool.stl"  scale="0.001 0.001 0.001"/>
+          <mesh filename="package://tht_robot_env/meshes/camera_calib_A4_Tool.stl"  scale="0.001 0.001 0.001"/>
         </geometry>
       </collision>
@@ -358,11 +358,11 @@
 	</joint>
     <!-- including the workspace urdf -->
-    <xacro:include filename="$(find thtr_robot_env)/urdf/inc/workspaces/space2_desc.xacro" />
+    <xacro:include filename="$(find tht_robot_env)/urdf/inc/workspaces/space2_desc.xacro" />
     <xacro:space2 base="${prefix}base_link"/>
     <!--Here another xacro:include for fixed_camera-->
-    <xacro:include filename="$(find thtr_robot_env)/urdf/inc/cameras/fixed_camera_cameracalib.xacro"/>
+    <xacro:include filename="$(find tht_robot_env)/urdf/inc/cameras/fixed_camera_cameracalib.xacro"/>
     <xacro:fixed_cam base="${prefix}base_link"/>
     <!--Here another xacro:include for gripper_camera-->
-    <!--xacro:include filename="$(find thtr_robot_env)/urdf/inc/cameras/gripper_camera.xacro"/>
+    <!--xacro:include filename="$(find tht_robot_env)/urdf/inc/cameras/gripper_camera.xacro"/>
     <xacro:gripper_cam base="${prefix}wrist_3_link"/-->
   </xacro:macro>

File: src/tht_robot_env/urdf/ur_macro_pointer.xacro (robot description, xacro)
@@ -1,6 +1,6 @@
 <?xml version="1.0"?>
 <robot xmlns:xacro="http://wiki.ros.org/xacro">
-  <xacro:include filename="$(find thtr_robot_env)/urdf/inc/ur_transmissions.xacro" />
-  <xacro:include filename="$(find thtr_robot_env)/urdf/inc/ur_common.xacro" />
+  <xacro:include filename="$(find tht_robot_env)/urdf/inc/ur_transmissions.xacro" />
+  <xacro:include filename="$(find tht_robot_env)/urdf/inc/ur_common.xacro" />
   <xacro:macro name="ur_robot" params="
     prefix
@@ -322,5 +322,5 @@
         <origin xyz="0 0 0" rpy="0 0 0"/>
         <geometry>
-          <mesh filename="package://thtr_robot_env/meshes/pointer_tool.stl" scale="0.001 0.001 0.001"/>
+          <mesh filename="package://tht_robot_env/meshes/pointer_tool.stl" scale="0.001 0.001 0.001"/>
         </geometry>
         <material name="black"/>
@@ -329,5 +329,5 @@
         <origin xyz="0 0 0" rpy="0 0 0"/>
         <geometry>
-          <mesh filename="package://thtr_robot_env/meshes/pointer_tool.stl"  scale="0.001 0.001 0.001"/>
+          <mesh filename="package://tht_robot_env/meshes/pointer_tool.stl"  scale="0.001 0.001 0.001"/>
         </geometry>
       </collision>
@@ -358,11 +358,11 @@
 	</joint>
     <!-- including the workspace urdf -->
-    <xacro:include filename="$(find thtr_robot_env)/urdf/inc/workspaces/space2_desc.xacro" />
+    <xacro:include filename="$(find tht_robot_env)/urdf/inc/workspaces/space2_desc.xacro" />
     <xacro:space2 base="${prefix}base_link"/>
     <!--Here another xacro:include for fixed_camera-->
-    <xacro:include filename="$(find thtr_robot_env)/urdf/inc/cameras/fixed_camera_cameracalib.xacro"/>
+    <xacro:include filename="$(find tht_robot_env)/urdf/inc/cameras/fixed_camera_cameracalib.xacro"/>
     <xacro:fixed_cam base="${prefix}base_link"/>
     <!--Here another xacro:include for gripper_camera-->
-    <!--xacro:include filename="$(find thtr_robot_env)/urdf/inc/cameras/gripper_camera.xacro"/>
+    <!--xacro:include filename="$(find tht_robot_env)/urdf/inc/cameras/gripper_camera.xacro"/>
     <xacro:gripper_cam base="${prefix}wrist_3_link"/-->
   </xacro:macro>

Commit message: updated camera urdf for right orientation on cam

File: src/tht_robot_env/urdf/inc/cameras/fixed_camera.xacro (robot description, xacro)
@@ -27,4 +27,10 @@
       		<child link="OAK_camera" />
 	</joint>
+	<link name="OAK_camera_rot"/>
+    <joint name="OAK_to_rot" type="fixed">
+      <origin xyz="0 0 0" rpy="0 0 ${pi}"/>
+      <parent link="OAK_camera"/>
+      <child link="OAK_camera_rot"/>
+    </joint>
 	<link name="camera_stand2">
 		<visual>

Commit message: update physical robot description and cam info

File: src/tht_robot_env/urdf/inc/cameras/fixed_camera.xacro (robot description, xacro)
@@ -36,5 +36,5 @@
 		<visual>
 			<geometry>
-    				<cylinder radius="0.02" length="1.0"/>
+    				<cylinder radius="0.02" length="0.70"/>
     			</geometry>
     			<material name="black"/>
@@ -42,10 +42,10 @@
 		<collision>
 			<geometry>
-    				<cylinder radius="0.02" length="0.9"/>
+    				<cylinder radius="0.02" length="0.70"/>
     			</geometry>
 		</collision>
 	</link>
 	<joint name="stand2_to_camera" type="fixed">
-		<origin xyz="0 -0.5 0" rpy="-${pi/2.0} 0 0"/>
+		<origin xyz="0 -0.35 0" rpy="-${pi/2.0} 0 0"/>
       		<parent link="OAK_camera" />
       		<child link="camera_stand2" />
@@ -54,5 +54,5 @@
 		<visual>
 			<geometry>
-    			<cylinder radius="0.02" length="1.6"/>
+    			<cylinder radius="0.02" length="1.86"/>
     		</geometry>
     		<material name="black"/>
@@ -60,10 +60,10 @@
 		<collision>
 			<geometry>
-    			<cylinder radius="0.01" length="1.55"/>
+    			<cylinder radius="0.01" length="1.86"/>
     		</geometry>
 		</collision>
 	</link>
     <joint name="stand1_to_stand2" type="fixed">
-    	<origin xyz="0 -0.78 -0.49" rpy="${pi/2.0} 0 0"/>
+    	<origin xyz="0 -0.93 -0.35" rpy="${pi/2.0} 0 0"/>
       <parent link="camera_stand2" />
       <child link="camera_stand1" />

File: src/tht_robot_env/urdf/ur.urdf.cameracalib.xacro (robot description, xacro)
@@ -16,4 +16,5 @@
      safety_pos_margin="0.15"
      safety_k_position="20"
+     end_effector_type="$(arg end_effector_type)"
      />
 </robot>

File: src/tht_robot_env/urdf/ur_macro_cameracalib.xacro (robot description, xacro)
@@ -13,5 +13,6 @@
     safety_limits:=false
     safety_pos_margin:=0.15
-    safety_k_position:=20">
+    safety_k_position:=20
+    end_effector_type">
     <!-- Load configuration data from the provided .yaml files -->
     <xacro:read_model_data
@@ -317,26 +318,49 @@
     </joint>
 		<xacro:property name="offset" value="0"/>
-    <!-- ROS-Industrial 'tool0' frame - all-zeros tool frame -->
-    <link name="calib_board">
-      <visual>
-        <origin xyz="0 0 0" rpy="0 0 0"/>
-        <geometry>
-          <mesh filename="package://tht_robot_env/meshes/camera_calib_A4_Tool.stl" scale="0.001 0.001 0.001"/>
-        </geometry>
-        <material name="black"/>
-      </visual>
-      <collision>
-        <origin xyz="0 0 0" rpy="0 0 0"/>
-        <geometry>
-          <mesh filename="package://tht_robot_env/meshes/camera_calib_A4_Tool.stl"  scale="0.001 0.001 0.001"/>
-        </geometry>
-      </collision>
-    </link>
-    <joint name="tool0-calib" type="fixed">
-      <!-- default toolframe - X+ left, Y+ up, Z+ front -->
-      <origin xyz="0 ${offset} 0.0850" rpy="0 0 0"/>
-      <parent link="${prefix}tool0"/>
-      <child link="calib_board"/>
-    </joint>
+    <!-- VETLE TEST -->
+    <xacro:if value="${end_effector_type == 1}">
+      <link name="end_effector_1">
+        <visual>
+          <origin xyz="0 0 0" rpy="0 0 0"/>
+          <geometry>
+            <mesh filename="package://tht_robot_env/meshes/camera_calib_A4_Tool.stl" scale="0.001 0.001 0.001"/>
+          </geometry>
+          <material name="black"/>
+        </visual>
+        <collision>
+          <origin xyz="0 0 0" rpy="0 0 0"/>
+          <geometry>
+            <mesh filename="package://tht_robot_env/meshes/camera_calib_A4_Tool.stl"  scale="0.001 0.001 0.001"/>
+          </geometry>
+        </collision>
+      </link>
+      <joint name="end_effector_joint" type="fixed">
+        <parent link="tool0"/>
+        <origin xyz="0 0 0.0850" rpy="0 0 0"/>
+        <child link="end_effector_1"/>
+      </joint>
+    </xacro:if>
+    <xacro:if value="${end_effector_type == 2}">
+      <link name="end_effector_2">
+        <visual>
+          <origin xyz="0 0 0" rpy="0 0 0"/>
+          <geometry>
+            <mesh filename="package://tht_robot_env/meshes/pointer_tool.stl" scale="0.001 0.001 0.001"/>
+          </geometry>
+          <material name="white"/>
+        </visual>
+        <collision>
+          <origin xyz="0 0 0" rpy="0 0 0"/>
+          <geometry>
+            <mesh filename="package://tht_robot_env/meshes/pointer_tool.stl"  scale="0.001 0.001 0.001"/>
+          </geometry>
+        </collision>
+      </link>
+      <joint name="end_effector_joint" type="fixed">
+        <origin xyz="0 0 0.133" rpy="0 0 0"/>
+        <child link="end_effector_2"/>
+        <parent link="tool0"/>
+      </joint>
+    </xacro:if>
     <link name="ground">
 		<visual>
@@ -361,5 +385,5 @@
     <xacro:space2 base="${prefix}base_link"/>
     <!--Here another xacro:include for fixed_camera-->
-    <xacro:include filename="$(find tht_robot_env)/urdf/inc/cameras/fixed_camera_cameracalib.xacro"/>
+    <xacro:include filename="$(find tht_robot_env)/urdf/inc/cameras/fixed_camera.xacro"/>
     <xacro:fixed_cam base="${prefix}base_link"/>
     <!--Here another xacro:include for gripper_camera-->
