Commit message: ur3 workd with word link

File: src/tht_bachelor_ur_launch/urdf/inc/ur_macro.xacro (robot description, xacro)
@@ -46,4 +46,5 @@
   <xacro:macro name="ur_robot" params="
     prefix
+    parent
     joint_limits_parameters_file
     kinematics_parameters_file
@@ -62,4 +63,5 @@
       physical_parameters_file="${physical_parameters_file}"
       visual_parameters_file="${visual_parameters_file}"/>
+    <link name="world" />
     <!-- Add URDF transmission elements (for ros_control) -->
     <xacro:ur_arm_transmission prefix="${prefix}" hw_interface="${transmission_hw_interface}" />
@@ -207,4 +209,10 @@
       </xacro:cylinder_inertial>
     </link>
+    <!-- base_joint fixes base_link to the environment -->
+    <joint name="${prefix}base_joint" type="fixed">
+      <origin xyz="0 0 0.82" rpy="0 0 0" />
+      <parent link="${parent}" />
+      <child link="${prefix}base_link" />
+    </joint>
     <!-- joints: main serial chain -->
     <joint name="${prefix}base_link-base_link_inertia" type="fixed">
@@ -407,5 +415,5 @@
       </joint>
     </xacro:if>
-    <!-- <link name="ground">
+    <link name="ground">
 		<visual>
 			<geometry>
@@ -419,10 +427,10 @@
     			</geometry>
 		</collision>
-	</link> -->
-	<!-- <joint name="ground_to_world" type="fixed">
+	</link>
+	<joint name="ground_to_world" type="fixed">
 		<origin xyz="0 0 -0.2" rpy="0 0 0"/>
 		<parent link="world" />
     <child link="ground" />
-	</joint> -->
+	</joint>
     <!-- including the workspace urdf -->
     <xacro:include filename="$(find tht_robot_env)/urdf/inc/workspaces/space2_desc.xacro" />

File: src/tht_bachelor_ur_launch/urdf/ur.xacro (robot description, xacro)
@@ -20,4 +20,5 @@
    <xacro:ur_robot
      prefix=""
+     parent="$(arg parent_link)"
      joint_limits_parameters_file="$(arg joint_limit_params)"
      kinematics_parameters_file="$(arg kinematics_params)"

Commit message: update ws

File: src/tht_bachelor_ur_launch/urdf/inc/ur_macro.xacro (robot description, xacro)
@@ -376,5 +376,5 @@
           <origin xyz="0 0 0" rpy="0 0 0"/>
           <geometry>
-            <mesh filename="package://tht_robot_env/meshes/camera_calib_A4_Tool.stl" scale="0.001 0.001 0.001"/>
+            <mesh filename="package://tht_bachelor_ur_launch/meshes/camera_calib_A4_Tool.stl" scale="0.001 0.001 0.001"/>
           </geometry>
           <material name="black"/>
@@ -383,5 +383,5 @@
           <origin xyz="0 0 0" rpy="0 0 0"/>
           <geometry>
-            <mesh filename="package://tht_robot_env/meshes/camera_calib_A4_Tool.stl"  scale="0.001 0.001 0.001"/>
+            <mesh filename="package://tht_bachelor_ur_launch/meshes/camera_calib_A4_Tool.stl"  scale="0.001 0.001 0.001"/>
           </geometry>
         </collision>
@@ -398,5 +398,5 @@
           <origin xyz="0 0 0" rpy="0 0 0"/>
           <geometry>
-            <mesh filename="package://tht_robot_env/meshes/pointer_tool.stl" scale="0.001 0.001 0.001"/>
+            <mesh filename="package://tht_bachelor_ur_launch/meshes/pointer_tool.stl" scale="0.001 0.001 0.001"/>
           </geometry>
           <material name="white"/>
@@ -405,5 +405,5 @@
           <origin xyz="0 0 0" rpy="0 0 0"/>
           <geometry>
-            <mesh filename="package://tht_robot_env/meshes/pointer_tool.stl"  scale="0.001 0.001 0.001"/>
+            <mesh filename="package://tht_bachelor_ur_launch/meshes/pointer_tool.stl"  scale="0.001 0.001 0.001"/>
           </geometry>
         </collision>
@@ -434,11 +434,11 @@
 	</joint>
     <!-- including the workspace urdf -->
-    <xacro:include filename="$(find tht_robot_env)/urdf/inc/workspaces/space2_desc.xacro" />
+    <xacro:include filename="$(find tht_bachelor_ur_launch)/urdf/inc/workspaces/space2_desc.xacro" />
     <xacro:space2 base="${prefix}base_link"/>
     <!--Here another xacro:include for fixed_camera-->
-    <xacro:include filename="$(find tht_robot_env)/urdf/inc/cameras/fixed_camera.xacro"/>
+    <xacro:include filename="$(find tht_bachelor_ur_launch)/urdf/inc/cameras/fixed_camera.xacro"/>
     <xacro:fixed_cam base="${prefix}base_link"/>
     <!--Here another xacro:include for gripper_camera-->
-    <!--xacro:include filename="$(find tht_robot_env)/urdf/inc/cameras/gripper_camera.xacro"/>
+    <!--xacro:include filename="$(find tht_bachelor_ur_launch)/urdf/inc/cameras/gripper_camera.xacro"/>
     <xacro:gripper_cam base="${prefix}wrist_3_link"/-->
   </xacro:macro>

File: src/tht_bachelor_ur_launch/urdf/inc/workspaces/space2_desc.xacro (robot description, xacro)
@@ -28,6 +28,6 @@
     <xacro:support_box
     	name="robot_table"
-    	vis_size_xyz= "0.45 0.45 ${table['height']}"
-    	coll_size_xyz= "0.45 0.45 ${table['height']}"
+    	vis_size_xyz= "${table['side']} ${table['side']} ${table['height']}"
+    	coll_size_xyz= "${table['side']} ${table['side']} ${table['height']}"
     	box_col="grey" />
     <joint name="robot_table_to_world" type="fixed">

Commit message: fixed minor configs to ws and changed color table

File: src/tht_bachelor_ur_launch/urdf/inc/ur_macro.xacro (robot description, xacro)
@@ -211,5 +211,5 @@
     <!-- base_joint fixes base_link to the environment -->
     <joint name="${prefix}base_joint" type="fixed">
-      <origin xyz="0 0 0.82" rpy="0 0 0" />
+      <origin xyz="0 0 1.025" rpy="0 0 0" />
       <parent link="${parent}" />
       <child link="${prefix}base_link" />
@@ -335,26 +335,29 @@
     	<color rgba="0.5 0.5 0.5 1"/>
     </material>
-     <material name="darkgrey">
+    <material name="darkgrey">
     	<color rgba="0.1 0.1 0.1 1"/>
     </material>
-     <material name="green">
+    <material name="green">
     	<color rgba="0 1 0 1"/>
     </material>
-     <material name="red">
+    <material name="red">
     	<color rgba="1 0 0 1"/>
     </material>
-     <material name="silver">
+    <material name="silver">
     	<color rgba="0.75 0.75 0.75 1"/>
     </material>
-     <material name="gold">
+    <material name="gold">
     	<color rgba="1 0.843 0 1"/>
     </material>
-     <material name="beige">
+    <material name="beige">
     	<color rgba="0.861 0.861 0.763 1"/>
     </material>
-     <material name="brown">
+    <material name="brown">
     	<color rgba="0.588 0.294 0 1"/>
     </material>
-     <material name="umber">
+    <material name="table_brown">
+      <color rgba="0.6 0.4 0.2 1"/>
+    </material>
+    <material name="umber">
     	<color rgba="0.43 0.149 0.055 1"/>
     </material>
@@ -418,5 +421,5 @@
       </joint>
     </xacro:if>
-    <link name="ground">
+    <!-- <link name="ground">
 		<visual>
 			<geometry>
@@ -435,5 +438,5 @@
 		<parent link="world" />
     <child link="ground" />
-	</joint>
+	</joint> -->
     <!-- including the workspace urdf -->
     <xacro:include filename="$(find tht_bachelor_ur_launch)/urdf/inc/workspaces/space2_desc.xacro" />

File: src/tht_bachelor_ur_launch/urdf/inc/workspaces/space2_desc.xacro (robot description, xacro)
@@ -26,5 +26,5 @@
     	vis_size_xyz= "${table['height']} ${table['width']} ${table['length']}"
     	coll_size_xyz= "${table['height']} ${table['width']} ${table['length']}"
-    	box_col="black" />
+    	box_col="table_brown" />
     <joint name="table to world" type="fixed">
       <parent link="base_link" />

Commit message: update readme, calib_menu, collision board

File: src/tht_bachelor_ur_launch/urdf/inc/ur_macro.xacro (robot description, xacro)
@@ -409,5 +409,5 @@
         </visual>
         <collision>
-          <origin xyz="0 0 0" rpy="0 0 0"/>
+          <origin xyz="0.002 0.002 0.002" rpy="0 0 0"/>
           <geometry>
             <mesh filename="package://tht_bachelor_ur_launch/meshes/pointer_tool.stl"  scale="0.001 0.001 0.001"/>
