Commit message: Change to environment

File: src/tht_bachelor_ur_launch/urdf/inc/cameras/fixed_camera.xacro (robot description, xacro)
@@ -36,5 +36,5 @@
 		<visual>
 			<geometry>
-    				<cylinder radius="0.02" length="0.70"/>
+    				<cylinder radius="0.02" length="0.60"/>
     			</geometry>
     			<material name="black"/>
@@ -42,5 +42,5 @@
 		<collision>
 			<geometry>
-    				<cylinder radius="0.02" length="0.70"/>
+    				<cylinder radius="0.02" length="0.60"/>
     			</geometry>
 		</collision>
@@ -54,5 +54,5 @@
 		<visual>
 			<geometry>
-    			<cylinder radius="0.02" length="1.86"/>
+    			<cylinder radius="0.02" length="1.90"/>
     		</geometry>
     		<material name="black"/>
@@ -60,5 +60,5 @@
 		<collision>
 			<geometry>
-    			<cylinder radius="0.01" length="1.86"/>
+    			<cylinder radius="0.02" length="1.90"/>
     		</geometry>
 		</collision>

File: src/tht_bachelor_ur_launch/urdf/inc/workspaces/space2_desc.xacro (robot description, xacro)
@@ -35,4 +35,14 @@
       <child link="robot_table" />
       <origin xyz="0 0 -${table['height'] / 2.0}" rpy="0 0 0" />
+    </joint>
+    <xacro:support_box
+    	name="table"
+    	vis_size_xyz= "1.20 0.45 0.735"
+    	coll_size_xyz= "1.22 0.47 0.737"
+    	box_col="black" />
+    <joint name="table to world" type="fixed">
+      <parent link="base_link" />
+      <child link="table" />
+      <origin xyz="0 0.375 -0.57" rpy="0 0 0" />
     </joint>
         <!-- REVY -->

Commit message: added calib pos ur3 move menu

File: src/tht_bachelor_ur_launch/urdf/inc/cameras/fixed_camera.xacro (robot description, xacro)
@@ -33,5 +33,5 @@
       <child link="OAK_camera_rot"/>
     </joint>
-	<link name="camera_stand2">
+	<!-- <link name="camera_stand2">
 		<visual>
 			<geometry>
@@ -68,5 +68,5 @@
       <parent link="camera_stand2" />
       <child link="camera_stand1" />
-    </joint>
+    </joint>  -->
 </xacro:macro>
 </robot>

File: src/tht_bachelor_ur_launch/urdf/inc/ur_macro.xacro (robot description, xacro)
@@ -329,5 +329,8 @@
     	<color rgba="0.01 0.01 0.01 1"/>
     </material>
-     <material name="grey">
+    <material name="light_gray">
+    	<color rgba="0.8 0.8 0.8 1"/>
+    </material>
+    <material name="grey">
     	<color rgba="0.5 0.5 0.5 1"/>
     </material>
@@ -420,5 +423,5 @@
     				<box size="10 10 0.42"/>
     			</geometry>
-    			<material name="umber"/>
+    			<material name="light_gray"/>
 		</visual>
 		<collision>

File: src/tht_bachelor_ur_launch/urdf/inc/workspaces/space2_desc.xacro (robot description, xacro)
@@ -30,5 +30,5 @@
       <parent link="base_link" />
       <child link="table" />
-      <origin xyz="0 0.40 -0.295" rpy="0 0 0" />
+      <origin xyz="0 0.40 -${0.30+table['height'] / 2}" rpy="0 0 0" />
     </joint>
 </xacro:macro>

Commit message: big update

File: src/tht_bachelor_ur_launch/urdf/inc/cameras/fixed_camera.xacro (robot description, xacro)
@@ -7,5 +7,20 @@
   <xacro:property name="camera" value="${measurements['dimensions']}"/>
   <!-- measurements for camera coordinates-->
-  <xacro:property name="coords" value="${measurements['cam1_coords']}"/>
+  <xacro:property name="cam_translation" value="${measurements['translation']}"/>
+  <xacro:property name="cam_rotation" value="${measurements['rotation']}"/>
+<!-- computing quaternion to rpy -->
+<xacro:macro name="quaternion_to_rpy" params="qx qy qz qw">
+        <!-- See: https://en.wikipedia.org/wiki/Conversion_between_quaternions_and_Euler_angles#Source_code_2 -->
+        <xacro:property name="sinr_cosp" value="${2 * (qw * qx + qy * qz)}"/>
+        <xacro:property name="cosr_cosp" value="${1 - 2 * (qx * qx + qy * qy)}"/>
+        <xacro:property name="roll" value="${atan2(sinr_cosp, cosr_cosp)}" scope="parent"/>
+        <xacro:property name="sinp" value="${2 * (qw * qy - qz * qx)}"/>
+        <xacro:property name="pitch" value="${copysign(pi / 2, sinp) if fabs(sinp) >= 1 else asin(sinp)}"
+                        scope="parent"/>
+        <xacro:property name="siny_cosp" value="${2 * (qw * qz + qx * qy)}"/>
+        <xacro:property name="cosy_cosp" value="${1 - 2 * (qy * qy + qz * qz)}"/>
+        <xacro:property name="yaw" value="${atan2(siny_cosp, cosy_cosp)}" scope="parent"/>
+    </xacro:macro>
+<xacro:quaternion_to_rpy qx="${cam_rotation['x']}" qy="${cam_rotation['y']}" qz="${cam_rotation['z']}" qw="${cam_rotation['w']}"/>
 <xacro:macro name="fixed_cam" params="base">
 	<link name="OAK_camera">
@@ -23,14 +38,15 @@
 	</link>
 	<joint name="camera_to_world" type="fixed">
-		<origin xyz="${coords['x']} ${coords['y']} ${coords['z']}" rpy="${-pi} 0 0"/>
+		<origin xyz="${cam_translation['x']} ${cam_translation['y']} ${cam_translation['z']}"
+				rpy="${roll} ${pitch} ${yaw}"/>
 		<parent link="${base}" />
       		<child link="OAK_camera" />
 	</joint>
-	<link name="OAK_camera_rot"/>
+	<!-- <link name="OAK_camera_rot"/>
     <joint name="OAK_to_rot" type="fixed">
       <origin xyz="0 0 0" rpy="0 0 ${pi}"/>
       <parent link="OAK_camera"/>
       <child link="OAK_camera_rot"/>
-    </joint>
+    </joint> -->
 	<!-- <link name="camera_stand2">
 		<visual>

File: src/tht_bachelor_ur_launch/urdf/inc/workspaces/space2_desc.xacro (robot description, xacro)
@@ -32,5 +32,9 @@
     <parent link="${base}"  />
     <child link="table_top" />
-    <origin xyz="-0.03 0.30 -${0.29+table_top['height'] / 2}" rpy="0 0 0" />
+    <origin xyz="-0.03 0.30 -0.2949" rpy="0 0 0" />
+    <!-- world frame til base_link = 1.025 (z-axis)
+         world frame til bord (topp) = 0,7401
+         bordtopp høyde = 0,02
+         base_link til bord (origo) = 1,025-0,7401+0,02/2 = 0.2949 -->
   </joint>
   <!-- Creating the two cylindrical legs -->
