Commit message: added teach pendant holder to urdf

File: src/tht_bachelor_ur_launch/urdf/inc/workspaces/space2_desc.xacro (robot description, xacro)
@@ -68,4 +68,26 @@
     <origin xyz="0 0 0" rpy="0 0 1.5708" />
   </joint>
+  <!-- Controller holder base -->
+  <xacro:support_box
+    name="controller_holder_base"
+    vis_size_xyz="0.21 0.13 0.005"
+    coll_size_xyz="0.21 0.13 0.005"
+    box_col="grey" />
+  <joint name="controller_holder_to_base" type="fixed">
+    <parent link="robot_base" />
+    <child link="controller_holder_base" />
+    <origin xyz="${0.21/2} 0 ${robot_base['height'] / 2.0}" rpy="0 0 0" />
+  </joint>
+  <!-- Controller holder rot -->
+  <xacro:support_box
+    name="controller_holder_rot"
+    vis_size_xyz="0.25 0.36 0.02"
+    coll_size_xyz="0.25 0.36 0.02"
+    box_col="grey" />
+  <joint name="controller_holder_rot_to_base" type="fixed">
+    <parent link="controller_holder_base" />
+    <child link="controller_holder_rot" />
+    <origin xyz="0.2 0 -0.08" rpy="0 0.7854 0" />
+  </joint>
 </xacro:macro>
 </robot>

Commit message: changes to environemnt and movemenu

File: src/tht_bachelor_ur_launch/urdf/inc/workspaces/space2_desc.xacro (robot description, xacro)
@@ -30,7 +30,7 @@
       box_col="table_brown" />
   <joint name="table to world" type="fixed">
-    <parent link="base_link" />
+    <parent link="${base}"  />
     <child link="table_top" />
-    <origin xyz="0 0.40 -${0.29+table_top['height'] / 2}" rpy="0 0 0" />
+    <origin xyz="-0.03 0.30 -${0.29+table_top['height'] / 2}" rpy="0 0 0" />
   </joint>
   <!-- Creating the two cylindrical legs -->

Commit message: update readme, calibration script and workspace

File: src/tht_bachelor_ur_launch/urdf/inc/workspaces/space2_desc.xacro (robot description, xacro)
@@ -32,5 +32,5 @@
     <parent link="${base}"  />
     <child link="table_top" />
-    <origin xyz="-0.03 0.30 -0.2949" rpy="0 0 0" />
+    <origin xyz="0 ${table_top['width']/2+0.065} -0.2949" rpy="0 0 0" />
     <!-- world frame til base_link = 1.025 (z-axis)
          world frame til bord (topp) = 0,7401
